File: ASG1.sch (KiCad schematic (older format))
At the start: 36 parts, among them U1 TL431LP, U2 1602-I2C, U3 AD7523, U4 LM741, U5 LM741

Commit message: Initial working version
Parts:
- removed D1, D2: 6.8V, symbol Device:D_Zener
- removed R4: 10M, symbol Device:R
- removed R5: 4.5K, symbol Device:R
- removed R6: 3.5K, symbol Device:R
- removed U4, U5: LM741, symbol Amplifier_Operational:LM741
- added C9: 100pF, symbol Device:C
- added C? (x5): 0.1uF, symbol Device:C
- added R19: 7.5K, symbol Device:R
- added R20: 4.3K, symbol Device:R
- added R21: 15K, symbol Device:R
- added R23: 30K, symbol Device:R
- added U? (x2): LM741, symbol local:LM741alt
- gave numbers to parts that had none: 20
- renumbered C1 to C7, R1 to R15, R2 to R16, R3 to R17, U2 to U1, U3 to U2, U1 to U3
Connections:
- net labels added: +12V, -12V, 5VREF
- net labels removed: +9V, -9V, 5V
- wire segments 145 -> 154
Other:
- moved on the sheet: A1, C1, C2, C3, C4, C5, C6, C7, R1, R10, R11, R12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

Commit message: Fixed schematic annotations
Parts:
- gave numbers to parts that had none: 7
- renumbered C7 to C10, C9 to C12, C6 to C7, R15 to R13, R16 to R14, R17 to R15, R19 to R16, R21 to R17, R20 to R18, R23 to R19, SW3 to SW2, U3 to U4
